File: Schematic/zx2020.kicad_sch (KiCad schematic)
At the start: 26 parts, among them J1 Bus breakout, J2 Conn_01x02_Male, J3 Conn_01x02_Male, J4 Conn_01x02_Male, J5 PATA_CONN, SW1 , U1 74LS02, U2 628128 128x8k RAM, U3 NE555P, U4 Z80CPU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

Commit message: Update zx2020.kicad_sch
Parts:
- removed unit 5 of U1
- removed U7: 7400, Package_DIP:DIP-14_W7.62mm, symbol 74xx:7400
- removed U8: 74HCT00, Package_DIP:DIP-14_W7.62mm, symbol 74xx:74HCT00
- added C1, C4, C5, C6, C7, C8: (no value), symbol Device:C
- added unit 5 of U4
- added unit 3 of U5
- added unit 1 of U5
- added U6: (no value), symbol 74xx:74LS00
- added unit 5 of U7
- C2, C3: value 100nF -> (none)
- J2, J3, J4: value Conn_01x02_Male -> (none)
- U5: value 74LS00 -> (none)
- renumbered C1 to C9, U4 to U1, U6 to U3, U1 to U4, U1 to U7, U3 to U9
Connections:
- net +5V: now also U5.7 (GND), X1.1 (EN), C1.1, C4.1, C5.1, C6.1, C7.1, C8.1, U4.14 (VCC), U6.14 (VCC), U7.14 (VCC); no longer U5.14 (VCC)
- net A4: now also U5.10, U5.9; no longer U5.4, U5.5
- net A5: now also U5.4
- net A6: now also U6.1, U6.5
- net GND: now also U5.14 (VCC), C1.2, C4.2, C5.2, C6.2, C7.2, C8.2, U4.7 (GND), U6.7 (GND), U7.7 (GND); no longer U5.7 (GND)
- net IORQ: now also U5.5, U5.3
- net VDP/~{CSR}: now also U6.6
- net VDP/~{CSW}: now also U6.3
- net ~{A4}: now also U5.8; no longer U5.6
- net ~{CS0}: now also U5.6
- net ~{IORQ}: now also U5.1, U5.2
- net at U7.13: now also U6.2
- net at U7.10: now also U6.4
- no-connect marks 79 -> 78
Other:
- note removed: "PS/2 Keyboard"
- note removed: "Terminal"
- moved on the sheet: J2, J3, J4, U5B, U7C, U7D, X1
